File: esp32.kicad_sch (KiCad schematic)
At the start: 26 parts, among them J5 TC2030-IDC, J8 USB_C_Receptacle_USB2.0, J9 Conn_01x04, SW1 GT-TC029B-H025-L1N, SW2 GT-TC029B-H025-L1N, U11 RT9080-33GJ5, U12 ESP32-S3-WROOM-1, Y1 32.768kHz

Commit message: added new i2c connector, power connector, and supporting components
Parts:
- added D2: SS310, Diode_SMD:D_SMA, symbol lcsc:SS310_C85658
- added F2: 5v 1A, Fuse:Fuse_0603_1608Metric, symbol Device:Fuse_Small
- added J10: Conn_01x02, Connector_PinSocket_2.54mm:PinSocket_1x02_P2.54mm_Vertical, symbol Connector_Generic:Conn_01x02
- added J6: Conn_01x04, Connector_PinSocket_2.54mm:PinSocket_1x04_P2.54mm_Vertical, symbol Connector_Generic:Conn_01x04
- D1: now not fitted
- J9: footprint Connector_PinSocket_2.54mm:PinSocket_1x04_P2.54mm_Vertical_SMD_Pin1Right -> Connector_PinSocket_2.54mm:PinSocket_1x04_P2.54mm_Vertical
Connections:
- net 3V3: now also J6.2 (Pin_2)
- net GND: now also J10.2 (Pin_2), J6.1 (Pin_1)
- net SCL: now also J6.3 (Pin_3)
- net SDA: now also J6.4 (Pin_4)
- new net: D2.2, F2.2
- new net 5V_OUT: D2.1, J10.1 (Pin_1)
- new net VIN_M: F2.1
Other:
- note added: "I2C Header for 4.3 inch LCD"
- note added: "power for 4.3 inch LCD"
