File: power.kicad_sch (KiCad schematic)
At the start: 29 parts, among them J7 Conn_01x02, Q1 CSD17311Q5, Q2 CSD17311Q5, Q4 2N7002K, U10 DS4432U+, U8 INA260, U9 TPS40305

Commit message: added new i2c connector, power connector, and supporting components
Parts:
- added F1: 5v 5a, Fuse:Fuse_0603_1608Metric, symbol Device:Fuse_Small
Connections:
- net VIN: now also F1.1; no longer J7.1 (Pin_1), U8.1 (IN+), U8.12 (VBUS), U8.2 (IN+), U8.3 (IN+)
- new net VIN_FUSED: F1.2, J7.1 (Pin_1), U8.1 (IN+), U8.12 (VBUS), U8.2 (IN+), U8.3 (IN+)
