File: power.kicad_sch (KiCad schematic)
At the start: 30 parts, among them J7 Conn_01x02, Q1 CSD17311Q5, Q2 CSD17311Q5, Q4 2N7002K, U10 DS4432U+, U8 INA260, U9 TPS40305

Commit message: added sda and scl puulups
Parts:
- C38: footprint Capacitor_SMD:C_0805_2012Metric -> Capacitor_SMD:C_0402_1005Metric
Changed lines of the file:
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@@
 			)
 		)
-		(property "Footprint" "Capacitor_SMD:C_0805_2012Metric"
+		(property "Footprint" "Capacitor_SMD:C_0402_1005Metric"
 			(at 58.4962 44.45 0)
 			(effects
