File: bitaxeUltra.kicad_pcb (KiCad board)
At the start: 4 copper layers, 56.5 x 99.8 mm, 137 parts, among them J1 54-00164, J2 Conn_01x02, J3 Conn_01x05, J4 Conn_01x04, J5 TC2030-IDC, J7 Conn_01x02, J8 USB_C_Receptacle_USB2.0, J9 Conn_01x04, Q1 CSD17311Q5, Q2 CSD17311Q5, Q4 2N7002K, SW1 GT-TC029B-H025-L1N, SW2 GT-TC029B-H025-L1N, U1 25MHz, U10 DS4432U+, U11 RT9080-33GJ5, U12 ESP32-S3-WROOM-1, U14 BM1366_mode1, U2 TXB0104RGYR, U5 MCP1824T-1802E, U6 MCP1824T-0802E, U7 EMC2101, U8 INA260, U9 TPS40305, Y1 32.768kHz

Commit message: fixing DRC
Parts:
- added D2: SS310, Diode_SMD:D_SMA, F.Cu at (113.5, 49.6)
- added F1: 5v 5a, Fuse:Fuse_0603_1608Metric, B.Cu at (79.7, 75.1)
- added F2: 5v 1A, Fuse:Fuse_0603_1608Metric, F.Cu at (108.3, 55.3)
- added G***: LOGO, LOGO, B.Cu at (80.1, 117.0)
- added J10: Conn_01x02, Connector_PinSocket_2.54mm:PinSocket_1x02_P2.54mm_Vertical, B.Cu at (119.3, 49.4)
- added J6: Conn_01x04, Connector_PinSocket_2.54mm:PinSocket_1x04_P2.54mm_Vertical, B.Cu at (90.9, 50.3)
- J9: footprint Connector_PinSocket_2.54mm:PinSocket_1x04_P2.54mm_Vertical_SMD_Pin1Right -> Connector_PinSocket_2.54mm:PinSocket_1x04_P2.54mm_Vertical
- SW1, SW2: footprint bitaxe:SW_CS1213AGF260_CRS -> bitaxe:SW_TL3340AF160QG
- moved J9 3.82 mm to (87.3, 50.3)
- moved SW2 2.14 mm to (132.2, 112.7), turned to -90 degrees
- moved SW1 1.99 mm to (132.2, 104.4), turned to -90 degrees
- moved J2 1.22 mm to (80.5, 129.1)
- moved H5 0.43 mm to (125.8, 136.0)
Connections:
- J7 pad 1: /Power/VIN -> /Power/VIN_FUSED
- U8 pad 1: /Power/VIN -> /Power/VIN_FUSED
- U8 pad 12: /Power/VIN -> /Power/VIN_FUSED
- U8 pad 2: /Power/VIN -> /Power/VIN_FUSED
- U8 pad 3: /Power/VIN -> /Power/VIN_FUSED
Routing:
- net Net-(D2-Pad2): track 0.00 -> 6.71 mm
- net /Power/VIN_FUSED: track 0.00 -> 6.26 mm, vias 0 -> 4
- net /Power/VIN: track 6.26 -> 0.00 mm, vias 12 -> 8
- net /SCL: track 126.5 -> 131.9 mm
- net /ESP32/5V_OUT: track 0.00 -> 3.86 mm
- net /ESP32/EN: track 81.0 -> 84.2 mm
- net /ESP32/IO0: track 92.0 -> 95.2 mm
- net /5V: track 217.6 -> 220.5 mm
- net /SDA: track 128.0 -> 129.5 mm
- net /3V3: track 74.3 -> 75.8 mm, vias 15 -> 14
- net GND: track 148.3 -> 147.2 mm, vias 83 -> 86
- added copper zone on B.Cu, net /Power/VIN_FUSED
- added copper zone on F.Cu, net /Power/VIN_FUSED
Other:
- board text added: "5V_OUT GND"
- board text added: "GND 3V3 SCL SDA"
